File: ergogen/left/out/pcbs/left.kicad_pcb (KiCad board)
At the start: 2 copper layers, 115 x 95 mm, 46 parts

Commit message: feat: Add mounting hole to the left
Parts:
- added ?: , HOLE_M2_TH, F.Cu at (157.0, 135.0)
Changed lines of the file:
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@@
             (pad "" smd rect (at -3.7 -1.1 90) (size 0.9 0.9) (layers B.Cu B.Paste B.Mask))
         )
+    (module HOLE_M2_TH (layer F.Cu)
+      (at 157 135 0)
+      (pad "" np_thru_hole circle (at 0 0 90) (size 4.0 4.0) (drill 4.0) (layers *.Cu *.Mask F.SilkS) (clearance 0.3)))
   (gr_line (start 90 64.5) (end 205 64.5) (angle 90) (layer Edge.Cuts) (width 0.15))
 (gr_line (start 90 64.5) (end 90 121.5) (angle 90) (layer Edge.Cuts) (width 0.15))
